File: pinchito_uesc.kicad_sch (KiCad schematic)
At the start: 21 parts, among them J1 Conn_01x03_Pin, J2 Conn_01x03_Pin, Q1 AO6604_C709896, Q2 AO6604_C709896, Q3 AO6604_C709896, Q4 AO6604_C5182068, Q5 AO6604_C5182068, Q6 AO6604_C5182068, U1 EFM8BB21F16G-C-QFN20

Commit message: Bump design to new MOSFETs
Parts:
- removed Q1, Q2, Q3: AO6604_C709896, component_lib:TSOP-6_L3.0-W1.5-P0.95-LS2.8-BR, symbol easyeda2kicad:AO6604_C709896
- removed Q4, Q5, Q6: AO6604_C5182068, component_lib:SOT-23-6_L2.9-W1.6-P0.95-LS2.8-BL, symbol easyeda2kicad:AO6604_C5182068
- removed TP1, TP2: TestPoint, TestPoint:TestPoint_Pad_1.0x1.0mm, symbol Connector:TestPoint
- added J3: Prog, Connector_PinHeader_2.00mm:PinHeader_1x03_P2.00mm_Vertical, symbol Connector:Conn_01x03_Pin
- added Q1, Q2, Q3: AO6604, component_lib:TSOP-6_L3.0-W1.5-P0.95-LS2.8-BR, symbol easyeda2kicad:AO6604
- J1: value Conn_01x03_Pin -> Motor; footprint Connector_PinHeader_2.54mm:PinHeader_1x03_P2.54mm_Vertical -> Connector_PinHeader_2.00mm:PinHeader_1x03_P2.00mm_Vertical
- J2: value Conn_01x03_Pin -> Power; footprint Connector_PinHeader_2.54mm:PinHeader_1x03_P2.54mm_Vertical -> Connector_PinHeader_2.00mm:PinHeader_1x03_P2.00mm_Vertical
Connections:
- net C2CK: now also J3.3 (Pin_3)
- net C2D: now also J3.2 (Pin_2)
- net GND: now also J3.1 (Pin_1), Q1.5 (S1), Q2.5 (S1), Q3.5 (S1)
- net M_A: now also Q3.4 (D2), Q3.6 (D1)
- net M_B: now also Q1.4 (D2), Q1.6 (D1)
- net M_C: now also Q2.4 (D2), Q2.6 (D1)
- net VCC: now also Q1.2 (S2), Q2.2 (S2), Q3.2 (S2)
- net at U1.11 (P1.2): now also Q1.1 (G1)
- net at U1.10 (P1.3): now also Q1.3 (G2)
- net at U1.14 (P1.0): now also Q3.1 (G1)
- net at U1.13 (P1.1): now also Q3.3 (G2)
- net at U1.8 (P1.5): now also Q2.3 (G2)
- net at U1.9 (P1.4): now also Q2.1 (G1)
Other:
- moved on the sheet: J1
